Commit message: 阿克曼的模型底盘仿真初步完成

File: urdf/akm_robot_sim.xacro (robot description, xacro)
@@ -39,5 +39,5 @@
         <origin xyz="0 0 0" rpy="0 0 0" />
         <geometry>
-            <box size="0.751 0.5 0.15" />
+            <box size="${body_length} ${body_width} ${body_depth}" />
         </geometry>
     </visual>
@@ -45,5 +45,5 @@
         <origin xyz="0.0 0 0.0" rpy="0 0 0" />
         <geometry>
-            <box size="0.751 0.5 0.15" />
+            <box size="${body_length} ${body_width} ${body_depth}" />
         </geometry>
     </collision>
@@ -52,5 +52,5 @@
       <parent link="base_link" />
       <child link="chassis_link" />
-      <origin xyz="0.0 0.0 0.0" rpy="0 0 0" />
+      <origin xyz="0.0 0.0 ${body_depth}" rpy="0 0 0" />
   </joint>
   <!-- FRONT LEFT WHEEL -->
@@ -236,11 +236,9 @@
       <limit lower="-3.14159" upper="3.14159" effort="70" velocity="-1" />
   </joint>
-  <!-- akm底盘插件 -->
-  <!-- https://docs.ros.org/en/ros2_packages/rolling/api/gazebo_plugins/generated/classgazebo__plugins_1_1GazeboRosAckermannDrive.html#class-documentation -->
   <!-- IMU joint -->
   <joint name="imu_joint" type="fixed">
     <axis xyz="0 1 0" />
-    <origin xyz="0.12 0 0.125" rpy="0 0 0"/>
-    <parent link="base_link"/>
+    <origin xyz="${body_length/2 - 0.05/2} 0 ${body_depth/2+0.05/2}" rpy="0 0 0"/>
+    <parent link="chassis_link"/>
     <child link="imu_link"/>
   </joint>
@@ -268,4 +266,5 @@
     </inertial>
   </link>
+  <!-- 仿真插件描述 -->
   <!-- Gazebo插件设置相关 主要是给各个模块加上颜色，可忽略-->
   <gazebo reference="chassis_link">
@@ -274,21 +273,27 @@
     <mu2>0.5</mu2>
   </gazebo>
-  <gazebo reference="front_left_wheel_link">
-    <material>Gazebo/Red</material>
-    <mu1>0.5</mu1>
-    <mu2>0.5</mu2>
-  </gazebo>
-  <!--<gazebo reference="wheel_2">
+  <gazebo reference="fr_left_wheel_link">
     <material>Gazebo/Black</material>
-  </gazebo>
-  <gazebo reference="wheel_3">
-    <material>Gazebo/Red</material>
-  </gazebo>
-  <gazebo reference="wheel_4">
-    <material>Gazebo/Black</material>
-  </gazebo> -->
-  <!-- <gazebo reference="virtual_steer_link">
+    <mu1>150.0</mu1>
+    <mu2>10.0</mu2>
+  </gazebo>
+  <gazebo reference="fr_right_wheel_link">
+      <material>Gazebo/Black</material>
+      <mu1>150.0</mu1>
+      <mu2>10.0</mu2>
+  </gazebo>
+  <gazebo reference="re_left_wheel_link">
+      <material>Gazebo/Black</material>
+      <mu1>150.0</mu1>
+      <mu2>10.0</mu2>
+  </gazebo>
+  <gazebo reference="re_right_wheel_link">
+      <material>Gazebo/Black</material>
+      <mu1>150.0</mu1>
+      <mu2>10.0</mu2>
+  </gazebo>
+  <gazebo reference="virtual_steer_link">
     <material>Gazebo/Yellow</material>
-  </gazebo> -->
+  </gazebo>
   <gazebo reference="imu_link">
     <material>Gazebo/BuildingFrame</material>
@@ -297,28 +302,4 @@
     <material>Gazebo/LightBlueLaser</material>
   </gazebo>
-  <!-- Virtual Steering wheel -->
-  <!-- <link name="virtual_steer_link">
-      <visual>
-          <origin xyz="0.0 0.0 0.0" rpy="0.0 0.0 0.0" />
-          <geometry>
-              <box size="0.01 0.15 0.075" />
-          </geometry>
-          <material name="">
-              <color rgba="1.0 1.0 0.0 1" />
-          </material>
-      </visual>
-      <inertial>
-          <origin xyz="0.0 0.0 0.0" rpy="0.0 0.0 0.0" />
-          <mass value="0.001" />
-          <inertia ixx="0.0" ixy="0.0" ixz="0.0" iyy="0.0" iyz="0.0" izz="0.0" />
-      </inertial>
-  </link>
-  <joint name="virtual_steering_wheel_joint" type="revolute">
-      <origin xyz="-0.32 0.0 0.0" rpy="0.0 0.0 0.0" />
-      <parent link="base_link" />
-      <child link="virtual_steer_link" />
-      <axis xyz="-1 0 0" />
-      <limit lower="-3" upper="3" effort="200" velocity="20" />
-  </joint> -->
   <!-- mid360_imu plugin -->
   <!-- https://github.com/ros-simulation/gazebo_ros_pkgs/wiki/ROS-2-Migration:-IMU-Sensors -->
@@ -394,6 +375,93 @@
   <!-- Livox-Mid360  -->
   <xacro:include filename="$(find ros2_livox_simulation)/urdf/mid360.xacro" />
-  <xacro:mid360 name="livox_frame" parent="base_link" topic="/livox/lidar">
-    <origin xyz="0.12 0.0 0.175" rpy="0 0 0" />
+  <xacro:mid360 name="livox_frame" parent="imu_link" topic="/livox/lidar">
+    <origin xyz="0.0 0.0 0.05" rpy="0 0 0" />
   </xacro:mid360>
+  <gazebo>
+      <plugin name="gazebo_ros_joint_state_publisher"
+          filename="libgazebo_ros_joint_state_publisher.so">
+          <update_rate>100</update_rate>
+          <joint_name>fr_right_steer_joint</joint_name>
+          <joint_name>fr_right_wheel_joint</joint_name>
+          <joint_name>fr_left_steer_joint</joint_name>
+          <joint_name>fr_left_wheel_joint</joint_name>
+          <joint_name>re_right_wheel_joint</joint_name>
+          <joint_name>re_left_wheel_joint</joint_name>
+          <joint_name>virtual_steering_wheel_joint</joint_name>
+      </plugin>
+  </gazebo>
+  <gazebo>
+      <plugin name="gazebo_ros_joint_pose_trajectory"
+          filename="libgazebo_ros_joint_pose_trajectory.so">
+          <update_rate>2</update_rate>
+      </plugin>
+  </gazebo>
+  <!-- akm底盘插件 -->
+  <!-- https://docs.ros.org/en/ros2_packages/rolling/api/gazebo_plugins/generated/classgazebo__plugins_1_1GazeboRosAckermannDrive.html#class-documentation -->
+  <gazebo>
+        <plugin name='gazebo_ackermann_drive' filename='libgazebo_ros_ackermann_drive.so'>
+            <ros>
+                <!-- <namespace>ugv_gazebo_ackermann</namespace> -->
+                <remapping>cmd_vel:=cmd_vel</remapping>
+                <remapping>odom:=odom</remapping>
+                <remapping>distance:=distance</remapping>
+            </ros>
+            <update_rate>100.0</update_rate>
+            <!-- wheels -->
+            <front_left_joint>fr_left_wheel_joint</front_left_joint>
+            <front_right_joint>fr_right_wheel_joint</front_right_joint>
+            <rear_left_joint>re_left_wheel_joint</rear_left_joint>
+            <rear_right_joint>re_right_wheel_joint</rear_right_joint>
+            <left_steering_joint>fr_left_steer_joint</left_steering_joint>
+            <right_steering_joint>fr_right_steer_joint</right_steering_joint>
+            <steering_wheel_joint>virtual_steering_wheel_joint</steering_wheel_joint>
+            <!-- Max absolute steer angle for tyre in radians-->
+            <!-- Any cmd_vel angular z greater than this would be capped -->
+            <max_steer>0.383972</max_steer>
+            <!-- Max absolute steering angle of steering wheel -->
+            <max_steering_angle>1.570796</max_steering_angle>
+            <!-- Max absolute linear speed in m/s -->
+            <max_speed>5</max_speed>
+            <!-- PID tuning -->
+            <left_steering_pid_gain>1500 0 1</left_steering_pid_gain>
+            <left_steering_i_range>0 0</left_steering_i_range>
+            <right_steering_pid_gain>1500 0 1</right_steering_pid_gain>
+            <right_steering_i_range>0 0</right_steering_i_range>
+            <linear_velocity_pid_gain>1500 0 1</linear_velocity_pid_gain>
+            <linear_velocity_i_range>0 0</linear_velocity_i_range>
+            <!-- output -->
+            <publish_odom>true</publish_odom>
+            <publish_odom_tf>true</publish_odom_tf>     <!-- Don't pubslish this when using robot
+            localization -->
+            <publish_wheel_tf>false</publish_wheel_tf>  <!-- Don't publish this. It will override all
+            wheel frames to robot_base_frame parameter below.-->
+            <publish_distance>true</publish_distance>
+            <odometry_frame>odom</odometry_frame>
+            <robot_base_frame>base_footprint</robot_base_frame>
+        </plugin>
+  </gazebo>
+  <!-- Virtual Steering wheel -->
+  <link name="virtual_steer_link">
+      <visual>
+          <origin xyz="0.0 0.0 0.0" rpy="0.0 0.0 0.0" />
+          <geometry>
+              <box size="0.01 0.15 0.075" />
+          </geometry>
+          <material name="">
+              <color rgba="1.0 1.0 0.0 1" />
+          </material>
+      </visual>
+      <inertial>
+          <origin xyz="0.0 0.0 0.0" rpy="0.0 0.0 0.0" />
+          <mass value="0.001" />
+          <inertia ixx="0.0" ixy="0.0" ixz="0.0" iyy="0.0" iyz="0.0" izz="0.0" />
+      </inertial>
+  </link>
+  <joint name="virtual_steering_wheel_joint" type="revolute">
+      <origin xyz="${body_length/3}  0.0 ${body_depth/2 + 0.075/2}" rpy="0.0 0.0 0.0" />
+      <parent link="chassis_link" />
+      <child link="virtual_steer_link" />
+      <axis xyz="-1 0 0" />
+      <limit lower="-3" upper="3" effort="200" velocity="20" />
+  </joint>
 </robot>

Commit message: 更改friction damping 参数，使控制机器人线速度 达到 较精准的目标值， 目前还是存在较大误差

File: urdf/akm_robot_sim.xacro (robot description, xacro)
@@ -27,4 +27,11 @@
       <origin xyz="0.0 0.0 0.0" rpy="0 0 0" />
   </joint>
+  <!-- <link name="camera_init">
+  </link>
+  <joint name="livox_joint" type="fixed">
+      <parent link="livox_frame" />
+      <child link="camera_init" />
+      <origin xyz="0.0 0.0 0.0" rpy="0 0 0" />
+  </joint> -->
   <link name="chassis_link">
     <inertial>
@@ -110,5 +117,5 @@
       <child link="fr_left_wheel_link" />
       <axis xyz="0 0 -1" />
-      <dynamics friction="0.8" damping="0.5" />
+      <dynamics friction="0.03" damping="0.02" />
       <limit lower="-3.14159" upper="3.14159" effort="200" velocity="-1" />
   </joint>
@@ -163,5 +170,5 @@
       <child link="fr_right_wheel_link" />
       <axis xyz="0 0 1" />
-      <dynamics friction="0.8" damping="0.5" />
+      <dynamics friction="0.03" damping="0.02" />
       <limit lower="-3.14159" upper="3.14159" effort="200" velocity="-1" />
   </joint>
@@ -198,5 +205,5 @@
       <child link="re_left_wheel_link" />
       <axis xyz="0 0 -1" />
-      <dynamics friction="0.8" damping="0.5" />
+      <dynamics friction="0.03" damping="0.02" />
       <limit lower="-3.14159" upper="3.14159" effort="70" velocity="-1" />
   </joint>
@@ -233,5 +240,5 @@
       <child link="re_right_wheel_link" />
       <axis xyz="0 0 1" />
-      <dynamics friction="0.8" damping="0.5" />
+      <dynamics friction="0.03" damping="0.02" />
       <limit lower="-3.14159" upper="3.14159" effort="70" velocity="-1" />
   </joint>
@@ -416,7 +423,8 @@
             <right_steering_joint>fr_right_steer_joint</right_steering_joint>
             <steering_wheel_joint>virtual_steering_wheel_joint</steering_wheel_joint>
+            <wheel_radius>0.1</wheel_radius>
             <!-- Max absolute steer angle for tyre in radians-->
             <!-- Any cmd_vel angular z greater than this would be capped -->
-            <max_steer>0.383972</max_steer>
+            <max_steer>1.570796</max_steer> <!--0.383972-->
             <!-- Max absolute steering angle of steering wheel -->
             <max_steering_angle>1.570796</max_steering_angle>

Commit message: 增加阻尼和摩擦，减少底盘静止时的微小运动

File: urdf/akm_robot_sim.xacro (robot description, xacro)
@@ -27,9 +27,9 @@
       <origin xyz="0.0 0.0 0.0" rpy="0 0 0" />
   </joint>
-  <!-- <link name="camera_init">
+  <!-- <link name="body">
   </link>
   <joint name="livox_joint" type="fixed">
       <parent link="livox_frame" />
-      <child link="camera_init" />
+      <child link="body" />
       <origin xyz="0.0 0.0 0.0" rpy="0 0 0" />
   </joint> -->
@@ -117,5 +117,5 @@
       <child link="fr_left_wheel_link" />
       <axis xyz="0 0 -1" />
-      <dynamics friction="0.03" damping="0.02" />
+      <dynamics friction="0.8" damping="0.5" />
       <limit lower="-3.14159" upper="3.14159" effort="200" velocity="-1" />
   </joint>
@@ -170,5 +170,5 @@
       <child link="fr_right_wheel_link" />
       <axis xyz="0 0 1" />
-      <dynamics friction="0.03" damping="0.02" />
+      <dynamics friction="0.8" damping="0.5" />
       <limit lower="-3.14159" upper="3.14159" effort="200" velocity="-1" />
   </joint>
@@ -205,5 +205,5 @@
       <child link="re_left_wheel_link" />
       <axis xyz="0 0 -1" />
-      <dynamics friction="0.03" damping="0.02" />
+      <dynamics friction="0.8" damping="0.5" /> <!-- 增加阻尼和摩擦 -->
       <limit lower="-3.14159" upper="3.14159" effort="70" velocity="-1" />
   </joint>
@@ -240,5 +240,5 @@
       <child link="re_right_wheel_link" />
       <axis xyz="0 0 1" />
-      <dynamics friction="0.03" damping="0.02" />
+      <dynamics friction="0.8" damping="0.5" />  <!-- 增加阻尼和摩擦 -->
       <limit lower="-3.14159" upper="3.14159" effort="70" velocity="-1" />
   </joint>
@@ -440,5 +440,5 @@
             <!-- output -->
             <publish_odom>true</publish_odom>
-            <publish_odom_tf>true</publish_odom_tf>     <!-- Don't pubslish this when using robot
+            <publish_odom_tf>false</publish_odom_tf>     <!-- Don't pubslish this when using robot
             localization -->
             <publish_wheel_tf>false</publish_wheel_tf>  <!-- Don't publish this. It will override all

Commit message: add body->base_footprint link, adapt for fast-lio

File: urdf/akm_robot_sim.xacro (robot description, xacro)
@@ -20,4 +20,12 @@
     <origin xyz="0 0 0" rpy="0 0 0" />
   </link>
+  <!--适配fast-lio-->
+  <link name="body">
+  </link>
+  <joint name="body_joint" type="fixed">
+      <parent link="body" />
+      <child link="base_footprint" />
+      <origin xyz="0.0 0.0 0.0" rpy="0 0 0" />
+  </joint>
   <link name="base_link">
   </link>

Commit message: 修改 mid-360 安装位置

File: urdf/akm_robot_sim.xacro (robot description, xacro)
@@ -3,5 +3,5 @@
   <xacro:property name="body_mass" value="25.0" />
   <xacro:property name="body_width" value="0.5" />
-  <xacro:property name="body_length" value="0.751" />
+  <xacro:property name="body_length" value="0.720" />
   <xacro:property name="body_depth" value="0.15" />
   <xacro:property name="wheel_radius" value="0.1" />
@@ -27,4 +27,6 @@
       <child link="base_footprint" />
       <origin xyz="0.0 0.0 0.0" rpy="0 0 0" />
+      <!--<origin xyz="${body_length/2 - 0.05/2} ${-1*(body_width/2 - 0.05/2)} ${body_depth/2+0.05/2}" rpy="0 0 0"/>-->
+      <!--<origin xyz="${-1 * (body_length/2 - 0.05/2)} ${body_width/2 - 0.05/2} ${-1 * (body_depth/2+0.05/2)}" rpy="0 0 0"/>-->
   </joint>
   <link name="base_link">
@@ -254,5 +256,6 @@
   <joint name="imu_joint" type="fixed">
     <axis xyz="0 1 0" />
-    <origin xyz="${body_length/2 - 0.05/2} 0 ${body_depth/2+0.05/2}" rpy="0 0 0"/>
+    <!-- <origin xyz="${body_length/2 - 0.05/2} 0 ${body_depth/2+0.05/2}" rpy="0 0 0"/>--> <!-- 前部正中间 -->
+    <origin xyz="${body_length/2 - 0.05/2} ${-1*(body_width/2 - 0.05/2)} ${body_depth/2+0.05/2}" rpy="0 0 0"/> <!-- ${10*PI/180} 右前角 下俯10度， 注意需要同步修改body->base_footprint的tf关系，tf关系相反-->
     <parent link="chassis_link"/>
     <child link="imu_link"/>

Commit message: update akm_robot_sim.xacro

File: urdf/akm_robot_sim.xacro (robot description, xacro)
@@ -26,7 +26,6 @@
       <parent link="body" />
       <child link="base_footprint" />
-      <origin xyz="0.0 0.0 0.0" rpy="0 0 0" />
-      <!--<origin xyz="${body_length/2 - 0.05/2} ${-1*(body_width/2 - 0.05/2)} ${body_depth/2+0.05/2}" rpy="0 0 0"/>-->
-      <!--<origin xyz="${-1 * (body_length/2 - 0.05/2)} ${body_width/2 - 0.05/2} ${-1 * (body_depth/2+0.05/2)}" rpy="0 0 0"/>-->
+      <!-- <origin xyz="0.0 0.0 0.0" rpy="0 0 0" />   -->
+      <origin xyz="${-1*(body_length/2 - 0.05/2)} ${body_width/2 - 0.05/2} 0" rpy="0 0 0"/>
   </joint>
   <link name="base_link">
