Commit message: add livox_frame link

File: urdf/akm_robot.xacro (robot description, xacro)
@@ -284,4 +284,33 @@
     </inertial>
   </link>
+  <!--livox_frame link -->
+  <link name="livox_frame">
+    <collision>
+      <origin xyz="0 0 0" rpy="0 0 0"/>
+      <geometry>
+        <box size="0.05 0.05 0.05"/>
+      </geometry>
+    </collision>
+    <visual>
+      <origin xyz="0 0 0" rpy="0 0 0"/>
+      <geometry>
+        <box size="0.05 0.05 0.05"/>
+      </geometry>
+      <material name="blue">
+        <color rgba="0 0 1 1"/>
+      </material>
+    </visual>
+    <inertial>
+      <mass value="1e-2" />
+      <origin xyz="0 0 0" rpy="0 0 0"/>
+      <inertia ixx="1e-6" ixy="0" ixz="0" iyy="1e-6" iyz="0" izz="1e-6" />
+    </inertial>
+  </link>
+  <!-- livox frame joint -->
+  <joint name="livox_joint" type="fixed">
+    <origin xyz="0 0 0" rpy="0 0 0"/>
+    <parent link="imu_link"/>
+    <child link="livox_frame"/>
+  </joint>
   <!-- Virtual Steering wheel -->
   <link name="virtual_steer_link">

Commit message: update tf: body-> base_footprint; remove IMU joint, livox_frame joint

File: urdf/akm_robot.xacro (robot description, xacro)
@@ -26,6 +26,6 @@
       <parent link="body" />
       <child link="base_footprint" />
-      <origin xyz="0.0 0.0 0.0" rpy="0 0 0" />
-      <!--<origin xyz="${body_length/2 - 0.05/2} ${-1*(body_width/2 - 0.05/2)} ${body_depth/2+0.05/2}" rpy="0 0 0"/>-->
+      <!-- <origin xyz="0.0 0.0 0.0" rpy="0 0 0" />   -->
+      <origin xyz="${-1*(body_length/2 - 0.05/2)} ${body_width/2 - 0.05/2} ${-1*(body_depth/2+0.05/2)}" rpy="0 0 0"/>
       <!--<origin xyz="${-1 * (body_length/2 - 0.05/2)} ${body_width/2 - 0.05/2} ${-1 * (body_depth/2+0.05/2)}" rpy="0 0 0"/>-->
   </joint>
@@ -254,13 +254,14 @@
   </joint>
   <!-- IMU joint -->
-  <joint name="imu_joint" type="fixed">
+  <!-- <origin xyz="${body_length/2 - 0.05/2} 0 ${body_depth/2+0.05/2}" rpy="0 0 0"/>--> <!-- 前部正中间 -->
+  <!-- ${10*PI/180} 右前角 下俯10度， 注意需要同步修改body->base_footprint的tf关系，tf关系相反-->
+  <!-- <joint name="imu_joint" type="fixed">
     <axis xyz="0 1 0" />
-    <!-- <origin xyz="${body_length/2 - 0.05/2} 0 ${body_depth/2+0.05/2}" rpy="0 0 0"/>--> <!-- 前部正中间 -->
-    <origin xyz="${body_length/2 - 0.05/2} ${-1*(body_width/2 - 0.05/2)} ${body_depth/2+0.05/2}" rpy="0 0 0"/> <!-- ${10*PI/180} 右前角 下俯10度， 注意需要同步修改body->base_footprint的tf关系，tf关系相反-->
+    <origin xyz="${body_length/2 - 0.05/2} ${-1*(body_width/2 - 0.05/2)} ${body_depth/2+0.05/2}" rpy="0 0 0"/>
     <parent link="chassis_link"/>
     <child link="imu_link"/>
-  </joint>
+  </joint> -->
   <!-- IMU -->
-  <link name="imu_link">
+  <!-- <link name="imu_link">
     <collision>
       <origin xyz="0 0 0" rpy="0 0 0"/>
@@ -283,7 +284,7 @@
       <inertia ixx="1e-6" ixy="0" ixz="0" iyy="1e-6" iyz="0" izz="1e-6" />
     </inertial>
-  </link>
+  </link> -->
   <!--livox_frame link -->
-  <link name="livox_frame">
+  <!-- <link name="livox_frame">
     <collision>
       <origin xyz="0 0 0" rpy="0 0 0"/>
@@ -306,11 +307,11 @@
       <inertia ixx="1e-6" ixy="0" ixz="0" iyy="1e-6" iyz="0" izz="1e-6" />
     </inertial>
-  </link>
+  </link> -->
   <!-- livox frame joint -->
-  <joint name="livox_joint" type="fixed">
+  <!-- <joint name="livox_joint" type="fixed">
     <origin xyz="0 0 0" rpy="0 0 0"/>
     <parent link="imu_link"/>
     <child link="livox_frame"/>
-  </joint>
+  </joint> -->
   <!-- Virtual Steering wheel -->
   <link name="virtual_steer_link">

Commit message: add imu_link and livox_frame fixed joint

File: urdf/akm_robot.xacro (robot description, xacro)
@@ -256,12 +256,12 @@
   <!-- <origin xyz="${body_length/2 - 0.05/2} 0 ${body_depth/2+0.05/2}" rpy="0 0 0"/>--> <!-- 前部正中间 -->
   <!-- ${10*PI/180} 右前角 下俯10度， 注意需要同步修改body->base_footprint的tf关系，tf关系相反-->
-  <!-- <joint name="imu_joint" type="fixed">
+  <joint name="imu_joint" type="fixed">
     <axis xyz="0 1 0" />
     <origin xyz="${body_length/2 - 0.05/2} ${-1*(body_width/2 - 0.05/2)} ${body_depth/2+0.05/2}" rpy="0 0 0"/>
     <parent link="chassis_link"/>
     <child link="imu_link"/>
-  </joint> -->
+  </joint>
   <!-- IMU -->
-  <!-- <link name="imu_link">
+  <link name="imu_link">
     <collision>
       <origin xyz="0 0 0" rpy="0 0 0"/>
@@ -284,7 +284,7 @@
       <inertia ixx="1e-6" ixy="0" ixz="0" iyy="1e-6" iyz="0" izz="1e-6" />
     </inertial>
-  </link> -->
+  </link>
   <!--livox_frame link -->
-  <!-- <link name="livox_frame">
+  <link name="livox_frame">
     <collision>
       <origin xyz="0 0 0" rpy="0 0 0"/>
@@ -307,11 +307,11 @@
       <inertia ixx="1e-6" ixy="0" ixz="0" iyy="1e-6" iyz="0" izz="1e-6" />
     </inertial>
-  </link> -->
+  </link>
   <!-- livox frame joint -->
-  <!-- <joint name="livox_joint" type="fixed">
+  <joint name="livox_joint" type="fixed">
     <origin xyz="0 0 0" rpy="0 0 0"/>
     <parent link="imu_link"/>
     <child link="livox_frame"/>
-  </joint> -->
+  </joint>
   <!-- Virtual Steering wheel -->
   <link name="virtual_steer_link">

Commit message: modify joint link: base_link -> chassis_link

File: urdf/akm_robot.xacro (robot description, xacro)
@@ -28,5 +28,5 @@
       <!-- <origin xyz="0.0 0.0 0.0" rpy="0 0 0" />   -->
       <origin xyz="${-1*(body_length/2 - 0.05/2)} ${body_width/2 - 0.05/2} ${-1*(body_depth/2+0.05/2)}" rpy="0 0 0"/>
-      <!--<origin xyz="${-1 * (body_length/2 - 0.05/2)} ${body_width/2 - 0.05/2} ${-1 * (body_depth/2+0.05/2)}" rpy="0 0 0"/>-->
+      <!-- <origin xyz="${body_length/2 - 0.05/2} ${-1*(body_width/2 - 0.05/2)} ${body_depth/2+0.05/2}" rpy="0 0 0"/> -->
   </joint>
   <link name="base_link">
@@ -69,5 +69,5 @@
       <parent link="base_link" />
       <child link="chassis_link" />
-      <origin xyz="0.0 0.0 ${body_depth}" rpy="0 0 0" />
+      <origin xyz="0.0 0.0 0.0" rpy="0 0 0" />
   </joint>
   <!-- FRONT LEFT WHEEL -->

Commit message: update joint parameters

File: urdf/akm_robot.xacro (robot description, xacro)
@@ -10,4 +10,7 @@
   <xacro:property name="steering_mass" value="0.01" />
   <xacro:property name="PI" value="3.1415926"/>
+  <xacro:property name="mid360_length" value="0.065"/>
+  <xacro:property name="mid360_O_height" value="0.047"/>
+  <xacro:property name="mid360_height" value="0.060"/>
   <xacro:macro name="default_inertial" params="mass">
     <inertial>
@@ -27,6 +30,5 @@
       <child link="base_footprint" />
       <!-- <origin xyz="0.0 0.0 0.0" rpy="0 0 0" />   -->
-      <origin xyz="${-1*(body_length/2 - 0.05/2)} ${body_width/2 - 0.05/2} ${-1*(body_depth/2+0.05/2)}" rpy="0 0 0"/>
-      <!-- <origin xyz="${body_length/2 - 0.05/2} ${-1*(body_width/2 - 0.05/2)} ${body_depth/2+0.05/2}" rpy="0 0 0"/> -->
+      <origin xyz="${-1*(body_length/2 - mid360_length/2 - 0.03)} ${body_width/2 - mid360_length/2 - 0.025} ${-1*(body_depth/2 + mid360_O_height)}" rpy="0 0 0"/>
   </joint>
   <link name="base_link">
@@ -258,5 +260,5 @@
   <joint name="imu_joint" type="fixed">
     <axis xyz="0 1 0" />
-    <origin xyz="${body_length/2 - 0.05/2} ${-1*(body_width/2 - 0.05/2)} ${body_depth/2+0.05/2}" rpy="0 0 0"/>
+    <origin xyz="${body_length/2 - mid360_length/2 - 0.03} ${-1*(body_width/2 - mid360_length/2 - 0.025)} ${body_depth/2 + mid360_O_height}" rpy="0 0 0"/>
     <parent link="chassis_link"/>
     <child link="imu_link"/>
@@ -267,5 +269,5 @@
       <origin xyz="0 0 0" rpy="0 0 0"/>
       <geometry>
-        <box size="0.05 0.05 0.05"/>
+        <box size="mid360_length mid360_length mid360_height"/>
       </geometry>
     </collision>
@@ -273,5 +275,5 @@
       <origin xyz="0 0 0" rpy="0 0 0"/>
       <geometry>
-        <box size="0.05 0.05 0.05"/>
+        <box size="mid360_length mid360_length mid360_height"/>
       </geometry>
       <material name="green">
@@ -290,5 +292,5 @@
       <origin xyz="0 0 0" rpy="0 0 0"/>
       <geometry>
-        <box size="0.05 0.05 0.05"/>
+        <box size="mid360_length mid360_length mid360_height"/>
       </geometry>
     </collision>
@@ -296,5 +298,5 @@
       <origin xyz="0 0 0" rpy="0 0 0"/>
       <geometry>
-        <box size="0.05 0.05 0.05"/>
+        <box size="mid360_length mid360_length mid360_height"/>
       </geometry>
       <material name="blue">

Commit message: multi(two) livox mid360 lidars

File: urdf/akm_robot.xacro (robot description, xacro)
@@ -255,15 +255,15 @@
       <limit lower="-3.14159" upper="3.14159" effort="70" velocity="-1" />
   </joint>
-  <!-- IMU joint -->
+  <!-- front IMU joint -->
   <!-- <origin xyz="${body_length/2 - 0.05/2} 0 ${body_depth/2+0.05/2}" rpy="0 0 0"/>--> <!-- 前部正中间 -->
   <!-- ${10*PI/180} 右前角 下俯10度， 注意需要同步修改body->base_footprint的tf关系，tf关系相反-->
-  <joint name="imu_joint" type="fixed">
+  <joint name="front_imu_joint" type="fixed">
     <axis xyz="0 1 0" />
     <origin xyz="${body_length/2 - mid360_length/2 - 0.03} ${-1*(body_width/2 - mid360_length/2 - 0.025)} ${body_depth/2 + mid360_O_height}" rpy="0 0 0"/>
     <parent link="chassis_link"/>
-    <child link="imu_link"/>
+    <child link="imu_link_192_168_1_111"/>
   </joint>
   <!-- IMU -->
-  <link name="imu_link">
+  <link name="imu_link_192_168_1_111">
     <collision>
       <origin xyz="0 0 0" rpy="0 0 0"/>
@@ -287,6 +287,36 @@
     </inertial>
   </link>
-  <!--livox_frame link -->
-  <link name="livox_frame">
+  <!-- rear IMU joint -->
+  <joint name="rear_imu_joint" type="fixed">
+    <axis xyz="0 1 0" />
+    <origin xyz="${-1*(body_length/2 - mid360_length/2 - 0.01)} ${body_width/2 - mid360_length/2 - 0.045} ${body_depth/2 + mid360_O_height}" rpy="0 0 0"/>
+    <parent link="chassis_link"/>
+    <child link="imu_link_192_168_1_140"/>
+  </joint>
+  <!-- IMU -->
+  <link name="imu_link_192_168_1_140">
+    <collision>
+      <origin xyz="0 0 0" rpy="0 0 0"/>
+      <geometry>
+        <box size="mid360_length mid360_length mid360_height"/>
+      </geometry>
+    </collision>
+    <visual>
+      <origin xyz="0 0 0" rpy="0 0 0"/>
+      <geometry>
+        <box size="mid360_length mid360_length mid360_height"/>
+      </geometry>
+      <material name="green">
+        <color rgba="0 1 0 1"/>
+      </material>
+    </visual>
+    <inertial>
+      <mass value="1e-2" />
+      <origin xyz="0 0 0" rpy="0 0 0"/>
+      <inertia ixx="1e-6" ixy="0" ixz="0" iyy="1e-6" iyz="0" izz="1e-6" />
+    </inertial>
+  </link>
+  <!--front livox_frame link -->
+  <link name="livox_frame_192_168_1_111">
     <collision>
       <origin xyz="0 0 0" rpy="0 0 0"/>
@@ -310,9 +340,38 @@
     </inertial>
   </link>
-  <!-- livox frame joint -->
-  <joint name="livox_joint" type="fixed">
+  <!--front livox frame joint -->
+  <joint name="front_livox_joint" type="fixed">
     <origin xyz="0 0 0" rpy="0 0 0"/>
-    <parent link="imu_link"/>
-    <child link="livox_frame"/>
+    <parent link="imu_link_192_168_1_111"/>
+    <child link="livox_frame_192_168_1_111"/>
+  </joint>
+  <!--rear livox_frame link -->
+  <link name="livox_frame_192_168_1_140">
+    <collision>
+      <origin xyz="0 0 0" rpy="0 0 0"/>
+      <geometry>
+        <box size="mid360_length mid360_length mid360_height"/>
+      </geometry>
+    </collision>
+    <visual>
+      <origin xyz="0 0 0" rpy="0 0 0"/>
+      <geometry>
+        <box size="mid360_length mid360_length mid360_height"/>
+      </geometry>
+      <material name="blue">
+        <color rgba="0 0 1 1"/>
+      </material>
+    </visual>
+    <inertial>
+      <mass value="1e-2" />
+      <origin xyz="0 0 0" rpy="0 0 0"/>
+      <inertia ixx="1e-6" ixy="0" ixz="0" iyy="1e-6" iyz="0" izz="1e-6" />
+    </inertial>
+  </link>
+  <!--rear livox frame joint -->
+  <joint name="rear_livox_joint" type="fixed">
+    <origin xyz="0 0 0" rpy="0 0 3.14159"/>
+    <parent link="imu_link_192_168_1_140"/>
+    <child link="livox_frame_192_168_1_140"/>
   </joint>
   <!-- Virtual Steering wheel -->

Commit message: add fixed camera_link for testing

File: urdf/akm_robot.xacro (robot description, xacro)
@@ -399,3 +399,10 @@
       <limit lower="-3" upper="3" effort="200" velocity="20" />
   </joint>
+  <!-- fixed camera_link -->
+  <link name="camera_link"></link>
+  <joint name="camera_joint" type="fixed">
+    <origin xyz="${body_length/2} 0.0 0.8" rpy="0 0 0"/>
+    <parent link="chassis_link"/>
+    <child link="camera_link"/>
+  </joint>
 </robot>
